File: Hardware/KiCad/RykerConnect-REV02/RykerConnect.kicad_pcb (KiCad board)
At the start: 2 copper layers, 102 x 34 mm, 67 parts, among them J1 12V Power In, J2 USB_C_Receptacle_USB2.0_16P, J3 Display Connector, J4 Ambient Light Connector, U1 USBLC6-2SC6, U2 MCP9808_MSOP, U3 Analog Devices RTC DS3231MZ_V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, U4 ESP32-S3-WROOM-1, U5 LMR50410Y3FQDBVRQ1

Commit message: update pcb to schematics
Parts:
- BT1: value Battery_Cell -> Holders Linx CR2032
- L1: value L -> 4.7uH
Connections:
- J3 pad 5: CHIP_PU -> DSP_RES
- U4 pad 8: unconnected-(U4-IO15-Pad8) -> DSP_RES
Routing:
- net DSP_RES: track 0.00 -> 27.7 mm, vias 0 -> 2
- net CHIP_PU: track 120.6 -> 103.7 mm, vias 6 -> 4
- net GND: track 368.8 -> 385.5 mm, vias 242 -> 227
- net SCL: track 114.0 -> 115.0 mm
Other:
- outline, holes or cut-outs redrawn

Commit message: update rev 2
Other:
- board text removed: "ChaostheoryBOT"
